File: pcb/FuseBox/fusebox.brd (EAGLE design)
At the start: 160 x 100 mm, 103 parts, among them Q2 INFINEON_IRLB8721PBFINFINEON_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, U1 ESP32-DEVKITC-32D, U2 TEXAS_INSTRUMENTS_TPS563249DD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, U3 MAXIM_ELECTRONICS_MAX7221CWGM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, U4 TEXAS_INSTRUMENTS_ADS1015IDGS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, U5 TEXAS_INSTRUMENTS_PCF8574PWTE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, U6 TEXAS_INSTRUMENTS_PCF8574PWTE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

Commit message: change to 2 layer
Routing:
- net GND: vias 57 -> 56
- net +5V: vias 3 -> 6
- added copper zone on layer 16, net +3V3
- removed copper zone on layer 15, net +3V3
- removed copper zone on layer 2, net GND

Commit message: minor GND plane fixes
Routing:
- net GND: track 44.2 -> 45.3 mm, vias 56 -> 54
Changed lines of the file:
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@@
 <?xml version="1.0" encoding="utf-8"?>
 <!DOCTYPE eagle SYSTEM "eagle.dtd">
-<eagle version="9.5.2">
+<eagle version="9.5.0">
 <drawing>
 <settings>
@@
 <via x="21.2725" y="55.88" extent="1-16" drill="0.35"/>
 <via x="21.2725" y="60.96" extent="1-16" drill="0.35"/>
-<wire x1="79.975" y1="65.5" x2="81" y2="65.5" width="0.254" layer="1"/>
-<wire x1="79.975" y1="64.5" x2="81" y2="64.5" width="0.254" layer="1"/>
-<via x="81" y="64.5" extent="1-16" drill="0.25"/>
-<via x="81" y="65.5" extent="1-16" drill="0.25"/>
 <wire x1="86.5" y1="67.5" x2="86.5" y2="68.5" width="0.254" layer="1"/>
 <via x="86.5" y="68.5" extent="1-16" drill="0.25"/>
@@
 <vertex x="159.5" y="0.5"/>
 </polygon>
-<wire x1="79.975" y1="65.5" x2="79.975" y2="64.5" width="0" layer="19" extent="1-1"/>
+<wire x1="79.975" y1="64.5" x2="79.01" y2="64.5" width="0.254" layer="1"/>
+<wire x1="79.01" y1="64.5" x2="78.74" y2="64.77" width="0.254" layer="1"/>
+<wire x1="78.74" y1="64.77" x2="78.74" y2="65.0875" width="0.254" layer="1"/>
+<wire x1="79.1525" y1="65.5" x2="78.74" y2="65.0875" width="0.254" layer="1"/>
+<wire x1="79.1525" y1="65.5" x2="79.975" y2="65.5" width="0.254" layer="1"/>
 </signal>
 <signal name="POTI_0">
